File: pcb/HACKPAD_V1.kicad_pcb (KiCad board)
At the start: 2 copper layers, 32 parts, among them X1 SW_Push, Y1 SW_Push

Commit message: pcb update
Routing:
- net 3.3v: track 237.1 -> 0.02 mm
- net view_button: track 11.1 -> 0.00 mm
Changed lines of the file:
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@@
-	)
-	(segment
-		(start 125.88 55)
-		(end 114.75 55)
-		(width 0.2)
-		(layer "B.Cu")
-		(net 11)
 	)
 	(segment
@@
 	)
 	(segment
-		(start 135.88 145.38)
-		(end 134 143.5)
-		(width 0.2)
-		(layer "B.Cu")
-		(net 27)
-	)
-	(segment
-		(start 118 65)
-		(end 119 66)
-		(width 0.2)
-		(layer "B.Cu")
-		(net 27)
-	)
-	(segment
-		(start 110.74 82.38)
-		(end 103.62 89.5)
-		(width 0.2)
-		(layer "B.Cu")
-		(net 27)
-	)
-	(segment
-		(start 139 135)
-		(end 134 135)
-		(width 0.2)
-		(layer "B.Cu")
-		(net 27)
-	)
-	(segment
-		(start 144 145.38)
-		(end 135.88 145.38)
-		(width 0.2)
-		(layer "B.Cu")
-		(net 27)
-	)
-	(segment
-		(start 134 135)
-		(end 126.5 135)
-		(width 0.2)
-		(layer "B.Cu")
-		(net 27)
-	)
-	(segment
-		(start 141.62 132.38)
-		(end 139 135)
-		(width 0.2)
-		(layer "B.Cu")
-		(net 27)
-	)
-	(segment
 		(start 121.015 70.985)
 		(end 121 71)
 		(width 0.2)
 		(layer "B.Cu")
-		(net 27)
-	)
-	(segment
-		(start 72 67.5)
-		(end 74.5 65)
-		(width 0.2)
-		(layer "B.Cu")
-		(net 27)
-	)
-	(segment
-		(start 74.5 65)
-		(end 118 65)
-		(width 0.2)
-		(layer "B.Cu")
-		(net 27)
-	)
-	(segment
-		(start 135.5 70.985)
-		(end 125.5 70.985)
-		(width 0.2)
-		(layer "B.Cu")
-		(net 27)
-	)
-	(segment
-		(start 141.62 77.105)
-		(end 141.62 111)
-		(width 0.2)
-		(layer "B.Cu")
-		(net 27)
-	)
-	(segment
-		(start 73.62 69.12)
-		(end 72 67.5)
-		(width 0.2)
-		(layer "B.Cu")
-		(net 27)
-	)
-	(segment
-		(start 135.5 70.985)
-		(end 141.62 77.105)
-		(width 0.2)
-		(layer "B.Cu")
-		(net 27)
-	)
-	(segment
-		(start 141.12 55)
-		(end 141.12 69.105)
-		(width 0.2)
-		(layer "B.Cu")
-		(net 27)
-	)
-	(segment
-		(start 116.5 73.5)
-		(end 110.74 73.5)
-		(width 0.2)
-		(layer "B.Cu")
-		(net 27)
-	)
-	(segment
-		(start 119 71)
-		(end 116.5 73.5)
-		(width 0.2)
-		(layer "B.Cu")
-		(net 27)
-	)
-	(segment
-		(start 110.74 73.5)
-		(end 110.74 82.38)
-		(width 0.2)
-		(layer "B.Cu")
-		(net 27)
-	)
-	(segment
-		(start 141.62 111)
-		(end 141.62 132.38)
-		(width 0.2)
-		(layer "B.Cu")
-		(net 27)
-	)
-	(segment
-		(start 134 143.5)
-		(end 134 135)
-		(width 0.2)
-		(layer "B.Cu")
-		(net 27)
-	)
-	(segment
-		(start 119 66)
-		(end 119 71)
-		(width 0.2)
-		(layer "B.Cu")
-		(net 27)
-	)
-	(segment
-		(start 151.8 70.985)
-		(end 143 70.985)
-		(width 0.2)
-		(layer "B.Cu")
-		(net 27)
-	)
-	(segment
-		(start 143 70.985)
-		(end 135.5 70.985)
-		(width 0.2)
-		(layer "B.Cu")
-		(net 27)
-	)
-	(segment
-		(start 141.12 69.105)
-		(end 143 70.985)
-		(width 0.2)
-		(layer "B.Cu")
-		(net 27)
-	)
-	(segment
-		(start 121 71)
-		(end 119 71)
-		(width 0.2)
-		(layer "B.Cu")
-		(net 27)
-	)
-	(segment
-		(start 125.5 70.985)
-		(end 121.015 70.985)
-		(width 0.2)
-		(layer "B.Cu")
-		(net 27)
-	)
-	(segment
-		(start 73.62 73.235)
-		(end 73.62 69.12)
-		(width 0.2)
-		(layer "B.Cu")

Commit message: updated pcb
Parts:
- moved R6 15.6 mm to (248.6, 105.5)
- moved RIGHT_JOYSTICK 9.04 mm to (185.5, 143.5)
- moved R12 5.22 mm to (249.0, 73.5)
- moved R11 3.59 mm to (214.9, 73.2)
- moved R1_TRIGGER 3.59 mm to (241.5, 72.0)
- moved R2_TRIGGER 3.59 mm to (237.7, 72.0)
- moved R9 3.38 mm to (61.8, 73.2)
- moved LEFT_JOYSTICK 0.94 mm to (144.8, 143.4)
- moved A_BUTTON 0.25 mm to (225.5, 130.5)
- moved B_BUTTON 0.25 mm to (242.8, 116.0)
- moved R5 0.25 mm to (203.6, 97.0)
- moved R7 0.25 mm to (203.5, 135.0)
- moved R8 0.25 mm to (187.1, 115.0)
- moved X_BUTTON 0.25 mm to (208.5, 116.0)
- moved Y_BUTTON 0.25 mm to (225.5, 101.5)
- renumbered A1 to A_BUTTON, B1 to B_BUTTON, Dpad_down1 to DPAD_DOWN, Dpad_left1 to DPAD_LEFT, Dpad_right1 to DPAD_RIGHT, Dpad_up1 to DPAD_UP, L1 to L1_TRIGGER, L2 to L2_TRIGGER, left_joystick1 to LEFT_JOYSTICK, Menu_button1 to MENU_BUTTON, R11 to R10, R13 to R11, R10 to R12, R12 to R13, R15 to R14, R1_trigger1 to R1_TRIGGER, R2_trigger1 to R2_TRIGGER, R6 to R5, R8 to R6, R5 to R8, right_joystick1 to RIGHT_JOYSTICK, TP4056_module1 to TP4056_MODULE, view_button1 to VIEW_BUTTON, X1 to X_BUTTON, Y1 to Y_BUTTON
Routing:
- net 3.3v: track 0.02 -> 120.5 mm
- net Dpad_right: track 0.00 -> 10.3 mm

Commit message: updated pcb
Parts:
- R1, R10, R11, R12, R13, R14, R2, R3, R4, R5, R6, R7, R8, R9: footprint Resistor_THT:R_Axial_DIN0614_L14.3mm_D5.7mm_P15.24mm_Horizontal -> Resistor_SMD:R_1206_3216Metric_Pad1.30x1.75mm_HandSolder
- moved R9 46.4 mm to (108.2, 74.5)
- moved R10 33.2 mm to (128.7, 74.5)
- moved L1_TRIGGER 32.0 mm to (116.0, 72.0)
- moved L2_TRIGGER 32.0 mm to (120.7, 72.0)
- moved R1_TRIGGER 30.7 mm to (210.8, 72.5)
- moved R2_TRIGGER 30.7 mm to (207.0, 72.5)
- moved R12 30.5 mm to (218.5, 75.0)
- moved R7 30.0 mm to (232.8, 128.5)
- moved R5 29.2 mm to (232.7, 99.5)
- moved R8 28.7 mm to (215.8, 114.0)
- moved R4 22.4 mm to (81.2, 114.0)
- moved MENU_BUTTON 20.8 mm to (201.8, 50.5)
- moved R11 16.0 mm to (199.0, 75.0)
- moved A_BUTTON 15.0 mm to (238.8, 123.5)
- moved B_BUTTON 15.0 mm to (256.0, 109.0)
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Routing:
- net 3.3v: track 120.5 -> 0.00 mm
- net Dpad_up: track 15.6 -> 0.00 mm
- net Dpad_right: track 10.3 -> 0.38 mm

Commit message: pcb
Parts:
- moved B_BUTTON 30.8 mm to (225.2, 109.5)
- moved Y_BUTTON 30.8 mm to (208.0, 95.0)
- moved A_BUTTON 30.5 mm to (208.2, 124.0)
- moved R5 30.5 mm to (202.2, 100.0)
- moved R6 30.5 mm to (219.2, 114.5)
- moved R7 30.5 mm to (202.3, 129.0)
- moved R8 30.5 mm to (185.3, 114.5)
- moved X_BUTTON 30.5 mm to (191.2, 109.5)
- moved DPAD_DOWN 28.5 mm to (108.2, 124.0)
- moved DPAD_LEFT 28.5 mm to (91.2, 109.5)
- moved DPAD_RIGHT 28.5 mm to (125.2, 109.5)
- moved DPAD_UP 28.5 mm to (108.2, 95.0)
- moved R1 28.5 mm to (127.2, 100.0)
- moved R3 28.5 mm to (126.8, 129.0)
- moved R4 28.5 mm to (109.8, 114.5)
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
Commit message: symbols and footprint
Parts:
- removed DPAD_DOWN, DPAD_LEFT, DPAD_RIGHT, DPAD_UP: SW_Push, Button_Switch_THT:SW_PUSH-12mm
- removed Doit_ESP32_DEVKITV1: ~, HACKPAD_V1:Doit_ESP32_DEVKITV1
- removed LEFT_JOYSTICK: Conn_01x05_Pin, Connector_PinSocket_2.54mm:PinSocket_1x05_P2.54mm_Vertical
- removed R1, R2, R3, R4: 4k7, Resistor_SMD:R_1206_3216Metric_Pad1.30x1.75mm_HandSolder
- removed TP4056_MODULE: ~, HACKPAD_V1:TP4056
- added ESP32_DEVKITV1: ~, HACKPAD_V1_FOOTPRINTS:ESP32_DEVKITV1, F.Cu at (165.1, 83.8)
- added J1: Conn_01x04_Pin, Connector_PinHeader_2.54mm:PinHeader_1x04_P2.54mm_Vertical, F.Cu at (132.1, 85.1)
- added J2: Conn_01x04_Pin, Connector_PinHeader_2.54mm:PinHeader_1x04_P2.54mm_Vertical, F.Cu at (127.0, 85.1)
- added J3: Conn_01x04_Pin, Connector_PinHeader_2.54mm:PinHeader_1x04_P2.54mm_Vertical, F.Cu at (150.3, 144.8)
- added J4: Conn_01x04_Pin, Connector_PinHeader_2.54mm:PinHeader_1x04_P2.54mm_Vertical, F.Cu at (154.9, 144.8)
- added TP4056_MODULE1: ~, HACKPAD_V1_FOOTPRINTS:TP4056, F.Cu at (156.1, 53.9)
- moved L1_TRIGGER1 0.69 mm to (104.2, 65.4)
- renumbered A_BUTTON to A_BUTTON1, B_BUTTON to B_BUTTON1, L1_TRIGGER to L1_TRIGGER1, L2_TRIGGER to L2_TRIGGER1, MENU_BUTTON to MENU_BUTTON1, R1_TRIGGER to R1_TRIGGER1, R2_TRIGGER to R2_TRIGGER1, RIGHT_JOYSTICK to RIGHT_JOYSTICK1, VIEW_BUTTON to VIEW_BUTTON1, X_BUTTON to X_BUTTON1, Y_BUTTON to Y_BUTTON1

Commit message: ADDED CODE
Parts:
- moved J3 14.8 mm to (137.6, 137.2)
- moved J4 14.8 mm to (142.2, 137.2)
- moved A_BUTTON1 10.5 mm to (215.9, 116.8)
- moved B_BUTTON1 10.5 mm to (232.9, 102.3)
- moved R5 10.5 mm to (209.8, 92.8)
- moved R6 10.5 mm to (226.9, 107.3)
- moved X_BUTTON1 10.5 mm to (198.9, 102.3)
- moved Y_BUTTON1 10.5 mm to (215.7, 87.8)
- moved R7 10.5 mm to (209.9, 121.8)
- moved R8 10.5 mm to (192.9, 107.3)
- moved RIGHT_JOYSTICK1 6.73 mm to (183.5, 147.3)
- moved L2_TRIGGER1 1.58 mm to (106.7, 66.0)
- moved R10 1.58 mm to (114.7, 68.5)
- moved R9 1.58 mm to (94.2, 68.5)
- moved L1_TRIGGER1 1.58 mm to (102.7, 66.0)
Routing:
- net 3.3v: track 0.00 -> 6.41 mm
Changed lines of the file:
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@@
 	(footprint "Connector_PinHeader_2.54mm:PinHeader_1x02_P2.54mm_Vertical"
 		(layer "F.Cu")
-		(at 104.18832 65.4455)
+		(at 102.71832 66.0255)
 		(descr "Through hole straight pin header, 1x02, 2.54mm pitch, single row")
 		(tags "Through hole pin header THT 1x02 2.54mm single row")
@@
 	(footprint "Button_Switch_THT:SW_PUSH-12mm"
 		(layer "F.Cu")
-		(at 191.25 109.5)
+		(at 198.9 102.34)
 		(descr "Generic SW PUSH 12mm, e.g https://sten-eswitch-13110800-production.s3.amazonaws.com/system/asset/product_line/data_sheet/143/TL1100.pdf")
 		(tags "tact sw push 12mm")
@@
 	(footprint "Connector_PinHeader_2.54mm:PinHeader_1x04_P2.54mm_Vertical"
 		(layer "F.Cu")
-		(at 150.29 144.78)
+		(at 137.59 137.16)
 		(descr "Through hole straight pin header, 1x04, 2.54mm pitch, single row")
 		(tags "Through hole pin header THT 1x04 2.54mm single row")
@@
 	(footprint "Button_Switch_THT:SW_PUSH-12mm"
 		(layer "F.Cu")
-		(at 208 95)
+		(at 215.65 87.84)
 		(descr "Generic SW PUSH 12mm, e.g https://sten-eswitch-13110800-production.s3.amazonaws.com/system/asset/product_line/data_sheet/143/TL1100.pdf")
 		(tags "tact sw push 12mm")
@@
 	(footprint "Resistor_SMD:R_1206_3216Metric_Pad1.30x1.75mm_HandSolder"
 		(layer "F.Cu")
-		(at 202.3 129)
+		(at 209.95 121.84)
 		(descr "Resistor SMD 1206 (3216 Metric), square (rectangular) end terminal, IPC_7351 nominal with elongated pad for handsoldering. (Body size source: IPC-SM-782 page 72, https://www.pcb-3d.com/wordpress/wp-content/uploads/ipc-sm-782a_amendment_1_and_2.pdf), generated with kicad-footprint-generator")
 		(tags "resistor handsolder")
@@
 	(footprint "Connector_PinSocket_2.54mm:PinSocket_1x05_P2.54mm_Vertical"
 		(layer "F.Cu")
-		(at 183.475 154.05 180)
+		(at 183.475 147.32 180)
 		(descr "Through hole straight socket strip, 1x05, 2.54mm pitch, single row (from Kicad 4.0.7), script generated")
 		(tags "Through hole socket strip THT 1x05 2.54mm single row")
@@
 	(footprint "Resistor_SMD:R_1206_3216Metric_Pad1.30x1.75mm_HandSolder"
 		(layer "F.Cu")
-		(at 116.15 67.96)
+		(at 114.68 68.54)
 		(descr "Resistor SMD 1206 (3216 Metric), square (rectangular) end terminal, IPC_7351 nominal with elongated pad for handsoldering. (Body size source: IPC-SM-782 page 72, https://www.pcb-3d.com/wordpress/wp-content/uploads/ipc-sm-782a_amendment_1_and_2.pdf), generated with kicad-footprint-generator")
 		(tags "resistor handsolder")
@@
 	(footprint "Connector_PinHeader_2.54mm:PinHeader_1x02_P2.54mm_Vertical"
 		(layer "F.Cu")
-		(at 108.15 65.46)
+		(at 106.68 66.04)
 		(descr "Through hole straight pin header, 1x02, 2.54mm pitch, single row")
 		(tags "Through hole pin header THT 1x02 2.54mm single row")
@@
 	(footprint "Button_Switch_THT:SW_PUSH-12mm"
 		(layer "F.Cu")
-		(at 208.25 124)
+		(at 215.9 116.84)
 		(descr "Generic SW PUSH 12mm, e.g https://sten-eswitch-13110800-production.s3.amazonaws.com/system/asset/product_line/data_sheet/143/TL1100.pdf")
 		(tags "tact sw push 12mm")
@@
 	(footprint "Resistor_SMD:R_1206_3216Metric_Pad1.30x1.75mm_HandSolder"
 		(layer "F.Cu")
-		(at 95.65 67.96)
+		(at 94.18 68.54)
 		(descr "Resistor SMD 1206 (3216 Metric), square (rectangular) end terminal, IPC_7351 nominal with elongated pad for handsoldering. (Body size source: IPC-SM-782 page 72, https://www.pcb-3d.com/wordpress/wp-content/uploads/ipc-sm-782a_amendment_1_and_2.pdf), generated with kicad-footprint-generator")
 		(tags "resistor handsolder")
@@
 	(footprint "Resistor_SMD:R_1206_3216Metric_Pad1.30x1.75mm_HandSolder"
 		(layer "F.Cu")
-		(at 202.2 100)
+		(at 209.85 92.84)
 		(descr "Resistor SMD 1206 (3216 Metric), square (rectangular) end terminal, IPC_7351 nominal with elongated pad for handsoldering. (Body size source: IPC-SM-782 page 72, https://www.pcb-3d.com/wordpress/wp-content/uploads/ipc-sm-782a_amendment_1_and_2.pdf), generated with kicad-footprint-generator")
 		(tags "resistor handsolder")
@@
 	(footprint "Resistor_SMD:R_1206_3216Metric_Pad1.30x1.75mm_HandSolder"
 		(layer "F.Cu")
-		(at 219.25 114.5)
+		(at 226.9 107.34)
 		(descr "Resistor SMD 1206 (3216 Metric), square (rectangular) end terminal, IPC_7351 nominal with elongated pad for handsoldering. (Body size source: IPC-SM-782 page 72, https://www.pcb-3d.com/wordpress/wp-content/uploads/ipc-sm-782a_amendment_1_and_2.pdf), generated with kicad-footprint-generator")
 		(tags "resistor handsolder")
@@
 	(footprint "Button_Switch_THT:SW_PUSH-12mm"
 		(layer "F.Cu")
-		(at 225.25 109.5)
+		(at 232.9 102.34)
 		(descr "Generic SW PUSH 12mm, e.g https://sten-eswitch-13110800-production.s3.amazonaws.com/system/asset/product_line/data_sheet/143/TL1100.pdf")
 		(tags "tact sw push 12mm")
@@
 	(footprint "Resistor_SMD:R_1206_3216Metric_Pad1.30x1.75mm_HandSolder"
 		(layer "F.Cu")
-		(at 185.3 114.5)
+		(at 192.95 107.34)
 		(descr "Resistor SMD 1206 (3216 Metric), square (rectangular) end terminal, IPC_7351 nominal with elongated pad for handsoldering. (Body size source: IPC-SM-782 page 72, https://www.pcb-3d.com/wordpress/wp-content/uploads/ipc-sm-782a_amendment_1_and_2.pdf), generated with kicad-footprint-generator")
 		(tags "resistor handsolder")
@@
 	(footprint "Connector_PinHeader_2.54mm:PinHeader_1x04_P2.54mm_Vertical"
 		(layer "F.Cu")
-		(at 154.94 144.78)
+		(at 142.24 137.16)
 		(descr "Through hole straight pin header, 1x04, 2.54mm pitch, single row")
 		(tags "Through hole pin header THT 1x04 2.54mm single row")
@@
 		)
 	)
+	(dimension
+		(type aligned)
+		(layer "F.Cu")
+		(pts
+			(xy 142.24 142.24) (xy 172.72 142.24)
+		)
+		(height -2.54)
+		(gr_text "30.4800 mm"
+			(at 157.48 137.9 0)
+			(layer "F.Cu")
+			(effects
+				(font
+					(size 1.5 1.5)
+					(thickness 0.3)
+				)
+			)
+		)
+		(format
+			(prefix "")
+			(suffix "")
+			(units 3)
+			(units_format 1)
+			(precision 4)
+		)
+		(style
+			(thickness 0.2)
+			(arrow_length 1.27)
+			(text_position_mode 0)
+			(extension_height 0.58642)
+			(extension_offset 0.5) keep_text_aligned)
+	)
+	(dimension
+		(type aligned)
+		(layer "F.Cu")
+		(pts
+			(xy 175.26 134.62) (xy 190.5 134.62)
+		)
+		(height 12.7)
+		(gr_text "15.2400 mm"
+			(at 182.88 145.52 0)
+			(layer "F.Cu")
+			(effects
+				(font
+					(size 1.5 1.5)
+					(thickness 0.3)
+				)
+			)
+		)
+		(format
+			(prefix "")
+			(suffix "")
+			(units 3)
+			(units_format 1)
+			(precision 4)
+		)
+		(style
+			(thickness 0.2)
+			(arrow_length 1.27)
+			(text_position_mode 0)
+			(extension_height 0.58642)
+			(extension_offset 0.5) keep_text_aligned)
+	)
 	(segment
-		(start 116.165 64.445)
-		(end 116.15 64.46)
+		(start 114.695 65.025)
+		(end 114.68 65.04)
 		(width 0.2)
 		(layer "B.Cu")
 		(net 2)
 	)
+	(segment
+		(start 154.94 73.385)
+		(end 154.94 76.2)
+		(width 0.2)
+		(layer "F.Cu")
+		(net 22)
+	)
+	(segment
+		(start 152.4 70.845)
+		(end 154.94 73.385)
+		(width 0.2)
+		(layer "F.Cu")
+		(net 22)
+	)
 )
