File: pcb/HACKPAD_V1.kicad_sch (KiCad schematic)
At the start: 31 parts

Commit message: PCB
Parts:
- removed Doit_ESP32_DEVKITV1: ~, GAME_PAD_ESP32:Doit_ESP32_DEVKITV1, symbol game_pad_esp32:Doit_esp32_devkitv1
- added Doit_ESP32_DEVKITV1: ~, HACKPAD_V1:Doit_ESP32_DEVKITV1, symbol HACKPAD_V1:Doit_esp32_devkitv1
- added TP4056_module1: ~, HACKPAD_V1:TP4056, symbol HACKPAD_V1:TP4056_module
- A1: renamed from A; footprint (none) -> Button_Switch_THT:SW_PUSH-12mm
- B1: renamed from B; footprint (none) -> Button_Switch_THT:SW_PUSH-12mm
- Dpad_down1: renamed from Dpad_down; footprint (none) -> Button_Switch_THT:SW_PUSH-12mm
- Dpad_left1: renamed from Dpad_left; footprint (none) -> Button_Switch_THT:SW_PUSH-12mm
- Dpad_right1: renamed from Dpad_right; footprint (none) -> Button_Switch_THT:SW_PUSH-12mm
- Dpad_up1: renamed from Dpad_up; footprint (none) -> Button_Switch_THT:SW_PUSH-12mm
- L1, L2: footprint (none) -> Connector_PinHeader_2.54mm:PinHeader_1x02_P2.54mm_Vertical
- Menu_button1: renamed from Menu_button; footprint (none) -> Button_Switch_THT:SW_PUSH-12mm
- R1, R10, R11, R12, R13, R15, R2, R3, R4, R5, R6, R7, R8, R9: footprint (none) -> Resistor_THT:R_Axial_DIN0614_L14.3mm_D5.7mm_P15.24mm_Horizontal
- R1_trigger1: renamed from R1; footprint (none) -> Connector_PinHeader_2.54mm:PinHeader_1x02_P2.54mm_Vertical
- R2_trigger1: renamed from R2; footprint (none) -> Connector_PinHeader_2.54mm:PinHeader_1x02_P2.54mm_Vertical
- X1: renamed from X; footprint (none) -> Button_Switch_THT:SW_PUSH-12mm
- Y1: renamed from Y; footprint (none) -> Button_Switch_THT:SW_PUSH-12mm
- left_joystick1: renamed from left_joystick; footprint (none) -> Connector_PinSocket_2.54mm:PinSocket_1x05_P2.54mm_Vertical
- right_joystick1: renamed from right_joystick; footprint (none) -> Connector_PinSocket_2.54mm:PinSocket_1x05_P2.54mm_Vertical
- view_button1: renamed from view_button; footprint (none) -> Button_Switch_THT:SW_PUSH-12mm
Connections:
- net A_button: now also Doit_ESP32_DEVKITV1.28 (D13)
- net B_button: now also Doit_ESP32_DEVKITV1.27 (D12)
- net Dpad_down: now also Doit_ESP32_DEVKITV1.4 (D02)
- net Dpad_left: now also Doit_ESP32_DEVKITV1.10 (D19)
- net Dpad_right: now also Doit_ESP32_DEVKITV1.9 (D18)
- net Dpad_up: now also Doit_ESP32_DEVKITV1.3 (D15)
- net L1: now also Doit_ESP32_DEVKITV1.11 (D21)
- net L2: now also Doit_ESP32_DEVKITV1.15 (D23)
- net Menu_button: now also Doit_ESP32_DEVKITV1.19 (D34)
- net R1: now also Doit_ESP32_DEVKITV1.24 (D26)
- net R2: now also Doit_ESP32_DEVKITV1.23 (D25)
- net SW-L: now also Doit_ESP32_DEVKITV1.14 (D22)
- net SW-R: now also Doit_ESP32_DEVKITV1.20 (D35)
- net VRx-L: now also Doit_ESP32_DEVKITV1.12 (RX0)
- net VRx-R: now also Doit_ESP32_DEVKITV1.22 (D33)
- net VRy-L: now also Doit_ESP32_DEVKITV1.5 (D04)
- net VRy-R: now also Doit_ESP32_DEVKITV1.21 (D32)
- net X_button: now also Doit_ESP32_DEVKITV1.25 (D27)
- net Y_button: now also Doit_ESP32_DEVKITV1.26 (D14)
- net view_button: now also Doit_ESP32_DEVKITV1.8 (D05)
- net +3V3 renamed 3.3v
- net 3.3v: now also left_joystick1.2 (Pin_2), right_joystick1.5 (Pin_5), Doit_ESP32_DEVKITV1.1 (3V3)
- net +5V renamed gnd
- net gnd: now also A1.1, B1.1, Dpad_down1.1, Dpad_left1.1, Dpad_right1.1, Dpad_up1.1, L1.1, L2.1, Menu_button1.1, R1_trigger1.1, R2_trigger1.1, X1.1, Y1.1, left_joystick1.1 (Pin_1), view_button1.1, Doit_ESP32_DEVKITV1.2 (GND); no longer left_joystick1.2 (Pin_2)
- removed net GND: A1.1, B1.1, Dpad_down1.1, Dpad_left1.1, Dpad_right1.1, Dpad_up1.1, L1.1, L2.1, Menu_button1.1, R1_trigger1.1, R2_trigger1.1, X1.1, Y1.1, left_joystick1.1 (Pin_1), right_joystick1.5 (Pin_5), view_button1.1
- new net: Doit_ESP32_DEVKITV1.29 (GND), TP4056_module1.OUT-
- new net: Doit_ESP32_DEVKITV1.30 (VIN), TP4056_module1.OUT+
- new net +BATT: TP4056_module1.B+
- new net -BATT: TP4056_module1.B-
- no-connect marks 0 -> 8
Other:
- moved on the sheet: left_joystick1, right_joystick1

Commit message: updated pcb
Parts:
- renumbered A1 to A_BUTTON, B1 to B_BUTTON, Dpad_down1 to DPAD_DOWN, Dpad_left1 to DPAD_LEFT, Dpad_right1 to DPAD_RIGHT, Dpad_up1 to DPAD_UP, L1 to L1_TRIGGER, L2 to L2_TRIGGER, left_joystick1 to LEFT_JOYSTICK, Menu_button1 to MENU_BUTTON, R11 to R10, R13 to R11, R10 to R12, R12 to R13, R15 to R14, R1_trigger1 to R1_TRIGGER, R2_trigger1 to R2_TRIGGER, R6 to R5, R8 to R6, R5 to R8, right_joystick1 to RIGHT_JOYSTICK, TP4056_module1 to TP4056_MODULE, view_button1 to VIEW_BUTTON, X1 to X_BUTTON, Y1 to Y_BUTTON
Connections:
- no-connect marks 8 -> 9
Changed lines of the file:
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@@
 	)
 	(no_connect
+		(at 33.02 20.32)
+	)
+	(no_connect
 		(at 161.29 60.96)
 	)
@@
 		(dnp no)
 		(fields_autoplaced yes)
-		(property "Reference" "R2_trigger1"
+		(property "Reference" "R2_TRIGGER"
 			(at 88.9 156.21 0)
 			(effects
@@
 			(project "DIY GAMEPAD(ESP32) WIRELESS"
 				(path "/29cb8219-b10d-47f3-b960-fd5b6212cd29"
-					(reference "R2_trigger1")
+					(reference "R2_TRIGGER")
 					(unit 1)
 				)
@@
 		(on_board yes)
 		(dnp no)
-		(property "Reference" "R12"
+		(property "Reference" "R13"
 			(at 58.166 182.118 90)
 			(effects
@@
 			(project "HACKPAD_V1"
 				(path "/29cb8219-b10d-47f3-b960-fd5b6212cd29"
-					(reference "R12")
+					(reference "R13")
 					(unit 1)
 				)
@@
 		(dnp no)
 		(fields_autoplaced yes)
-		(property "Reference" "B1"
+		(property "Reference" "B_BUTTON"
 			(at 88.9 105.41 0)
 			(effects
@@
 			(project "DIY GAMEPAD(ESP32) WIRELESS"
 				(path "/29cb8219-b10d-47f3-b960-fd5b6212cd29"
-					(reference "B1")
+					(reference "B_BUTTON")
 					(unit 1)
 				)
@@
 		(on_board yes)
 		(dnp no)
-		(property "Reference" "R13"
+		(property "Reference" "R11"
 			(at 100.076 157.988 90)
 			(effects
@@
 			(project "DIY GAMEPAD(ESP32) WIRELESS"
 				(path "/29cb8219-b10d-47f3-b960-fd5b6212cd29"
-					(reference "R13")
+					(reference "R11")
 					(unit 1)
 				)
@@
 		(dnp no)
 		(fields_autoplaced yes)
-		(property "Reference" "L2"
+		(property "Reference" "L2_TRIGGER"
 			(at 44.45 156.21 0)
 			(effects
@@
 			(project "DIY GAMEPAD(ESP32) WIRELESS"
 				(path "/29cb8219-b10d-47f3-b960-fd5b6212cd29"
-					(reference "L2")
+					(reference "L2_TRIGGER")
 					(unit 1)
 				)
@@
 		(dnp no)
 		(fields_autoplaced yes)
-		(property "Reference" "R1_trigger1"
+		(property "Reference" "R1_TRIGGER"
 			(at 88.9 144.78 0)
 			(effects
@@
 			(project "DIY GAMEPAD(ESP32) WIRELESS"
 				(path "/29cb8219-b10d-47f3-b960-fd5b6212cd29"
-					(reference "R1_trigger1")
+					(reference "R1_TRIGGER")
 					(unit 1)
 				)
@@
 		(dnp no)
 		(fields_autoplaced yes)
-		(property "Reference" "Dpad_left1"
+		(property "Reference" "DPAD_LEFT"
 			(at 44.45 54.61 0)
 			(effects
@@
 			(project "DIY GAMEPAD(ESP32) WIRELESS"
 				(path "/29cb8219-b10d-47f3-b960-fd5b6212cd29"
-					(reference "Dpad_left1")
+					(reference "DPAD_LEFT")
 					(unit 1)
 				)
@@
 		(dnp no)
 		(fields_autoplaced yes)
-		(property "Reference" "Menu_button1"
+		(property "Reference" "MENU_BUTTON"
 			(at 91.44 180.34 0)
 			(effects
@@
 			(project "HACKPAD_V1"
 				(path "/29cb8219-b10d-47f3-b960-fd5b6212cd29"
-					(reference "Menu_button1")
+					(reference "MENU_BUTTON")
 					(unit 1)
 				)
@@
 		(dnp no)
 		(fields_autoplaced yes)
-		(property "Reference" "Dpad_right1"
+		(property "Reference" "DPAD_RIGHT"
 			(at 88.9 54.61 0)
 			(effects
@@
 			(project "DIY GAMEPAD(ESP32) WIRELESS"
 				(path "/29cb8219-b10d-47f3-b960-fd5b6212cd29"
-					(reference "Dpad_right1")
+					(reference "DPAD_RIGHT")
 					(unit 1)
 				)
@@
 		(on_board yes)
 		(dnp no)
-		(property "Reference" "R6"
+		(property "Reference" "R5"
 			(at 77.216 91.948 90)
 			(effects
@@
 			(project "DIY GAMEPAD(ESP32) WIRELESS"
 				(path "/29cb8219-b10d-47f3-b960-fd5b6212cd29"
-					(reference "R6")
+					(reference "R5")
 					(unit 1)
 				)
@@
 		(dnp no)
 		(fields_autoplaced yes)
-		(property "Reference" "#PWR034"
+		(property "Reference" "#PWR0101"
 			(at 167.64 62.23 0)
 			(effects
@@
 			(project ""
 				(path "/29cb8219-b10d-47f3-b960-fd5b6212cd29"
-					(reference "#PWR034")
+					(reference "#PWR0101")
 					(unit 1)
 				)
@@
 		(dnp no)
 		(fields_autoplaced yes)
-		(property "Reference" "view_button1"
+		(property "Reference" "VIEW_BUTTON"
 			(at 46.99 180.34 0)
 			(effects
@@
 			(project "HACKPAD_V1"
 				(path "/29cb8219-b10d-47f3-b960-fd5b6212cd29"
-					(reference "view_button1")
+					(reference "VIEW_BUTTON")
 					(unit 1)
 				)
@@
 		(on_board yes)
 		(dnp no)
-		(property "Reference" "R10"
+		(property "Reference" "R12"
 			(at 100.076 146.558 90)
 			(effects
@@
 			(project "DIY GAMEPAD(ESP32) WIRELESS"
 				(path "/29cb8219-b10d-47f3-b960-fd5b6212cd29"
-					(reference "R10")
+					(reference "R12")
 					(unit 1)
 				)
@@
 		(dnp no)
 		(fields_autoplaced yes)
-		(property "Reference" "Dpad_up1"
+		(property "Reference" "DPAD_UP"
 			(at 66.04 39.37 0)
 			(effects
@@
 			(project ""
 				(path "/29cb8219-b10d-47f3-b960-fd5b6212cd29"
-					(reference "Dpad_up1")
+					(reference "DPAD_UP")
 					(unit 1)
 				)
@@
 		(on_board yes)
 		(dnp no)
-		(property "Reference" "R8"
+		(property "Reference" "R6"
 			(at 100.076 107.188 90)
 			(effects
@@
 			(project "DIY GAMEPAD(ESP32) WIRELESS"
 				(path "/29cb8219-b10d-47f3-b960-fd5b6212cd29"
-					(reference "R8")
+					(reference "R6")
 					(unit 1)
 				)
@@
 		(dnp no)
 		(fields_autoplaced yes)
-		(property "Reference" "A1"
+		(property "Reference" "A_BUTTON"
 			(at 69.85 118.11 0)
 			(effects
@@
 			(project "DIY GAMEPAD(ESP32) WIRELESS"
 				(path "/29cb8219-b10d-47f3-b960-fd5b6212cd29"
-					(reference "A1")
+					(reference "A_BUTTON")
 					(unit 1)
 				)
@@
 		(on_board yes)
 		(dnp no)
-		(property "Reference" "R5"
+		(property "Reference" "R8"
 			(at 55.626 107.188 90)
 			(effects
@@
 			(project "DIY GAMEPAD(ESP32) WIRELESS"
 				(path "/29cb8219-b10d-47f3-b960-fd5b6212cd29"
-					(reference "R5")
+					(reference "R8")
 					(unit 1)
 				)
@@
 		(dnp no)
 		(fields_autoplaced yes)
-		(property "Reference" "#PWR033"
+		(property "Reference" "#PWR0102"
 			(at 167.64 59.69 0)
 			(effects
@@
 			(project ""
 				(path "/29cb8219-b10d-47f3-b960-fd5b6212cd29"
-					(reference "#PWR033")
+					(reference "#PWR0102")
 					(unit 1)
 				)
@@
 		(dnp no)
 		(fields_autoplaced yes)
-		(property "Reference" "Y1"
+		(property "Reference" "Y_BUTTON"
 			(at 66.04 90.17 0)
 			(effects
@@
 			(project "DIY GAMEPAD(ESP32) WIRELESS"
 				(path "/29cb8219-b10d-47f3-b960-fd5b6212cd29"
-					(reference "Y1")
+					(reference "Y_BUTTON")
 					(unit 1)
 				)
@@
 		(dnp no)
 		(fields_autoplaced yes)
-		(property "Reference" "Dpad_down1"
+		(property "Reference" "DPAD_DOWN"
 			(at 69.85 67.31 0)
 			(effects
@@
 			(project "DIY GAMEPAD(ESP32) WIRELESS"
 				(path "/29cb8219-b10d-47f3-b960-fd5b6212cd29"
-					(reference "Dpad_down1")
+					(reference "DPAD_DOWN")
 					(unit 1)
 				)
@@
 		(dnp no)
 		(fields_autoplaced yes)
-		(property "Reference" "TP4056_module1"
-			(at 166.3803 54.61 0)
+		(property "Reference" "TP4056_MODULE"
+			(at 166.37 55.88 0)
 			(effects
 				(font
@@
 			(project ""
 				(path "/29cb8219-b10d-47f3-b960-fd5b6212cd29"
-					(reference "TP4056_module1")
+					(reference "TP4056_MODULE")
 					(unit 1)
 				)
@@
 		(on_board yes)
 		(dnp no)
-		(property "Reference" "left_joystick1"
+		(property "Reference" "LEFT_JOYSTICK"
 			(at 131.445 93.98 0)
 			(effects
@@
 			(project ""
 				(path "/29cb8219-b10d-47f3-b960-fd5b6212cd29"
-					(reference "left_joystick1")
+					(reference "LEFT_JOYSTICK")
 					(unit 1)
 				)
@@
 		(dnp no)
 		(fields_autoplaced yes)
-		(property "Reference" "X1"
+		(property "Reference" "X_BUTTON"
 			(at 44.45 105.41 0)
 			(effects
@@
 			(project "DIY GAMEPAD(ESP32) WIRELESS"
 				(path "/29cb8219-b10d-47f3-b960-fd5b6212cd29"
-					(reference "X1")
+					(reference "X_BUTTON")
 					(unit 1)
 				)
@@
 		(on_board yes)
 		(dnp no)
-		(property "Reference" "R11"
+		(property "Reference" "R10"
 			(at 55.626 157.988 90)
 			(effects
@@
 			(project "DIY GAMEPAD(ESP32) WIRELESS"
 				(path "/29cb8219-b10d-47f3-b960-fd5b6212cd29"
-					(reference "R11")
+					(reference "R10")
 					(unit 1)
 				)
@@
 		(dnp no)
 		(fields_autoplaced yes)
-		(property "Reference" "L1"
+		(property "Reference" "L1_TRIGGER"
 			(at 44.45 144.78 0)
 			(effects
@@
 			(project "DIY GAMEPAD(ESP32) WIRELESS"
 				(path "/29cb8219-b10d-47f3-b960-fd5b6212cd29"
-					(reference "L1")
+					(reference "L1_TRIGGER")
 					(unit 1)
 				)
@@
 		(on_board yes)
 		(dnp no)
-		(property "Reference" "R15"
+		(property "Reference" "R14"
 			(at 102.616 182.118 90)
 			(effects
@@
 			(project "HACKPAD_V1"
 				(path "/29cb8219-b10d-47f3-b960-fd5b6212cd29"
-					(reference "R15")
+					(reference "R14")
 					(unit 1)
 				)
@@
 		(on_board yes)
 		(dnp no)
-		(property "Reference" "right_joystick1"
+		(property "Reference" "RIGHT_JOYSTICK"
 			(at 163.576 93.98 0)
 			(effects
@@
 			(project "DIY GAMEPAD(ESP32) WIRELESS"
 				(path "/29cb8219-b10d-47f3-b960-fd5b6212cd29"
-					(reference "right_joystick1")
+					(reference "RIGHT_JOYSTICK")
 					(unit 1)
 				)

Commit message: pcb
Parts:
- added J2: Conn_01x04_Pin, symbol Connector:Conn_01x04_Pin
Changed lines of the file:
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@@
+	)
+	(symbol
+		(lib_id "Connector:Conn_01x04_Pin")
+		(at 34.29 72.39 0)
+		(unit 1)
+		(exclude_from_sim no)
+		(in_bom yes)
+		(on_board yes)
+		(dnp no)
+		(fields_autoplaced yes)
+		(property "Reference" "J2"
+			(at 34.925 64.77 0)
+			(effects
+				(font
+					(size 1.27 1.27)
+				)
+			)
+		)
+		(property "Value" "Conn_01x04_Pin"
+			(at 34.925 67.31 0)
+			(effects
+				(font
+					(size 1.27 1.27)
+				)
+			)
+		)
+		(property "Footprint" ""
+			(at 34.29 72.39 0)
+			(effects
+				(font
+					(size 1.27 1.27)
+				)
+				(hide yes)
+			)
+		)
+		(property "Datasheet" "~"
+			(at 34.29 72.39 0)
+			(effects
+				(font
+					(size 1.27 1.27)
+				)
+				(hide yes)
+			)
+		)
+		(property "Description" "Generic connector, single row, 01x04, script generated"
+			(at 34.29 72.39 0)
+			(effects
+				(font
+					(size 1.27 1.27)
+				)
+				(hide yes)
+			)
+		)
+		(pin "4"
+		)
+		(pin "2"
+		)
+		(pin "1"
+		)
+		(pin "3"
+		)
+		(instances
+			(project ""
+				(path "/29cb8219-b10d-47f3-b960-fd5b6212cd29"
+					(reference "J2")
+					(unit 1)
+				)
+			)
+		)
 	)
 	(symbol
@@
 		(on_board yes)
 		(dnp no)
-		(fields_autoplaced yes)
 		(property "Reference" "DPAD_DOWN"
 			(at 69.85 67.31 0)

Commit message: symbols and footprint
Parts:
- removed DPAD_DOWN, DPAD_LEFT, DPAD_RIGHT, DPAD_UP: SW_Push, Button_Switch_THT:SW_PUSH-12mm, symbol Switch:SW_Push
- removed Doit_ESP32_DEVKITV1: ~, HACKPAD_V1:Doit_ESP32_DEVKITV1, symbol HACKPAD_V1:Doit_esp32_devkitv1
- removed LEFT_JOYSTICK: Conn_01x05_Pin, Connector_PinSocket_2.54mm:PinSocket_1x05_P2.54mm_Vertical, symbol Connector:Conn_01x05_Pin
- removed R1, R2, R3, R4: 4k7, Resistor_THT:R_Axial_DIN0614_L14.3mm_D5.7mm_P15.24mm_Horizontal, symbol Device:R
- removed TP4056_MODULE: ~, HACKPAD_V1:TP4056, symbol HACKPAD_V1:TP4056_module
- added ESP32_DEVKITV1: ~, HACKPAD_V1_FOOTPRINTS:ESP32_DEVKITV1, symbol HACKPAD_V1_SYM:ESP32_DEVKITV1
- added J1, J3, J4: Conn_01x04_Pin, Connector_PinHeader_2.54mm:PinHeader_1x04_P2.54mm_Vertical, symbol Connector:Conn_01x04_Pin
- added TP4056_MODULE1: ~, HACKPAD_V1_FOOTPRINTS:TP4056, symbol HACKPAD_V1_SYM:TP4056
- J2: footprint (none) -> Connector_PinHeader_2.54mm:PinHeader_1x04_P2.54mm_Vertical
- R10, R11, R12, R13, R14, R5, R6, R7, R8, R9: footprint Resistor_THT:R_Axial_DIN0614_L14.3mm_D5.7mm_P15.24mm_Horizontal -> Resistor_SMD:R_1206_3216Metric_Pad1.30x1.75mm_HandSolder
- renumbered A_BUTTON to A_BUTTON1, B_BUTTON to B_BUTTON1, L1_TRIGGER to L1_TRIGGER1, L2_TRIGGER to L2_TRIGGER1, MENU_BUTTON to MENU_BUTTON1, R1_TRIGGER to R1_TRIGGER1, R2_TRIGGER to R2_TRIGGER1, RIGHT_JOYSTICK to RIGHT_JOYSTICK1, VIEW_BUTTON to VIEW_BUTTON1, X_BUTTON to X_BUTTON1, Y_BUTTON to Y_BUTTON1
Connections:
- net +BATT: now also TP4056_MODULE1.B+
- net -BATT: now also TP4056_MODULE1.B-
- net 3.3v: now also ESP32_DEVKITV1.1 (3V3), J1.4 (Pin_4), J4.4 (Pin_4)
- net A_button: now also ESP32_DEVKITV1.28 (D13)
- net B_button: now also ESP32_DEVKITV1.27 (D12)
- net Dpad_down: now also J2.1 (Pin_1), ESP32_DEVKITV1.4 (D02)
- net Dpad_left: now also J2.4 (Pin_4), ESP32_DEVKITV1.10 (D19)
- net Dpad_right: now also J2.3 (Pin_3), ESP32_DEVKITV1.9 (D18)
- net Dpad_up: now also J2.2 (Pin_2), ESP32_DEVKITV1.3 (D15)
- net L1: now also ESP32_DEVKITV1.11 (D21)
- net L2: now also ESP32_DEVKITV1.15 (D23)
- net Menu_button: now also ESP32_DEVKITV1.19 (D34)
- net R1: now also ESP32_DEVKITV1.24 (D26)
- net R2: now also ESP32_DEVKITV1.23 (D25)
- net SW-L: now also ESP32_DEVKITV1.14 (D22), J3.1 (Pin_1)
- net SW-R: now also ESP32_DEVKITV1.20 (D35)
- net VRx-L: now also ESP32_DEVKITV1.12 (RX0), J3.2 (Pin_2)
- net VRx-R: now also ESP32_DEVKITV1.22 (D33)
- net VRy-L: now also ESP32_DEVKITV1.5 (D04), J3.3 (Pin_3)
- net VRy-R: now also ESP32_DEVKITV1.21 (D32)
- net X_button: now also ESP32_DEVKITV1.25 (D27)
- net Y_button: now also ESP32_DEVKITV1.26 (D14)
- net gnd: now also ESP32_DEVKITV1.2 (GND), J1.3 (Pin_3), J4.3 (Pin_3)
- net view_button: now also ESP32_DEVKITV1.8 (D05)
- new net: ESP32_DEVKITV1.30 (VIN), TP4056_MODULE1.OUT+
- new net: ESP32_DEVKITV1.29 (GND), TP4056_MODULE1.OUT-
- no-connect marks 9 -> 10

Commit message: ADDED CODE
Changed lines of the file:
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@@
 		(dnp no)
 		(property "Reference" "J3"
-			(at 119.38 96.266 0)
+			(at 124.714 96.266 0)
 			(effects
 				(font
@@
 		)
 		(property "Value" "Conn_01x04_Pin"
-			(at 113.792 94.488 0)
+			(at 119.888 92.202 0)
 			(effects
 				(font
